File: hardware/stm32-rfid-clone.kicad_pcb (KiCad board)
At the start: 2 copper layers, 112 parts, among them J101 USB, M101 Mouting Hole, M102 Mouting Hole, M103 Mouting Hole, M104 Mouting Hole, P101 JTAG10, P102 BATTERY, P103 DEBUG, P104 READIND, P105 SPEAKER, P201 ANT, Q201 2N2222, Q202 2N2222, Q203 2N2907, U101 MOSFET-P, U102 STM32-48PIN, U103 AP6502, U104 MOSFET-N, U105 MIC2288, U201 TL084, X101 8MHz, X102 32.768kHz

Commit message: edge cuts
Parts:
- moved S103 2.00 mm to (128.0, 138.0)
Routing:
- net GNDPWR: track 67.4 -> 69.5 mm, vias 27 -> 28
- net /VIN: track 59.1 -> 60.4 mm
Other:
- board outline added: 61 x 61 mm
Changed lines of the file:
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@@
     (links 208)
     (no_connects 0)
-    (area 0 0 0 0)
+    (area 80.4478 75.353519 143.050001 148.628201)
     (thickness 1.6)
-    (drawings 0)
-    (tracks 804)
+    (drawings 4)
+    (tracks 811)
     (zones 0)
     (modules 112)
@@
   )
   (module stm32:CKCOMP-OS102011MA1QN1 (layer F.Cu)
-    (at 126 138)
+    (at 128 138)
     (fp_text reference S103 (at 0 -2.75) (layer F.SilkS)
       (effects (font (size 0.6 0.6) (thickness 0.1)))
@@
       (net 33 "Net-(C120-Pad1)"))
   )
+  (gr_line (start 81.28 139.7) (end 81.28 78.74) (angle 90) (layer Edge.Cuts) (width 0.1))
+  (gr_line (start 142.24 139.7) (end 81.28 139.7) (angle 90) (layer Edge.Cuts) (width 0.1))
+  (gr_line (start 142.24 78.74) (end 142.24 139.7) (angle 90) (layer Edge.Cuts) (width 0.1))
+  (gr_line (start 81.28 78.74) (end 142.24 78.74) (angle 90) (layer Edge.Cuts) (width 0.1))
   (segment (start 104.65 99.25) (end 104.05 99.25) (width 0.254) (layer F.Cu) (net 1))
   (segment (start 99.8 101.1) (end 102.8 101.1) (width 0.254) (layer F.Cu) (net 1))
@@
   (segment (start 94 89.55) (end 94 86.126) (width 0.254) (layer F.Cu) (net 19))
   (segment (start 94 86.126) (end 94.626 85.5) (width 0.254) (layer F.Cu) (net 19))
+  (segment (start 130 138) (end 130 137) (width 0.254) (layer B.Cu) (net 20))
+  (segment (start 126.55 135.55) (end 118.5 135.55) (width 0.254) (layer F.Cu) (net 20))
+  (segment (start 127 136) (end 126.55 135.55) (width 0.254) (layer F.Cu) (net 20))
+  (via (at 127 136) (size 0.889) (layers F.Cu B.Cu) (net 20))
+  (segment (start 129 136) (end 127 136) (width 0.254) (layer B.Cu) (net 20))
+  (segment (start 130 137) (end 129 136) (width 0.254) (layer B.Cu) (net 20))
+  (segment (start 118.5 135.55) (end 118.5 135.5) (width 0.254) (layer F.Cu) (net 20))
+  (segment (start 118.5 135.5) (end 118.5 135.55) (width 0.254) (layer F.Cu) (net 20))
+  (segment (start 130 138) (end 130 137) (width 0.254) (layer F.Cu) (net 20))
+  (segment (start 129.5 131) (end 132 128.5) (width 0.254) (layer F.Cu) (net 20))
+  (segment (start 129.5 136.5) (end 129.5 131) (width 0.254) (layer F.Cu) (net 20))
+  (segment (start 130 137) (end 129.5 136.5) (width 0.254) (layer F.Cu) (net 20))
   (segment (start 105.5 134) (end 106.4 134.9) (width 0.254) (layer F.Cu) (net 20))
-  (segment (start 105.5 134) (end 104.5 133) (width 0.254) (layer F.Cu) (net 20))
-  (segment (start 104.5 133) (end 104.5 132) (width 0.254) (layer F.Cu) (net 20))
-  (segment (start 103 128.05) (end 103.55 128.05) (width 0.254) (layer F.Cu) (net 20))
-  (segment (start 104.5 129) (end 103.55 128.05) (width 0.254) (layer F.Cu) (net 20))
-  (segment (start 104.5 132) (end 104.5 129) (width 0.254) (layer F.Cu) (net 20))
-  (segment (start 117.35 135.55) (end 118.5 135.55) (width 0.254) (layer F.Cu) (net 20))
-  (segment (start 116.7 134.9) (end 117.35 135.55) (width 0.254) (layer F.Cu) (net 20))
-  (via (at 116.7 134.9) (size 0.889) (layers F.Cu B.Cu) (net 20))
-  (segment (start 106.4 134.9) (end 116.7 134.9) (width 0.254) (layer B.Cu) (net 20))
   (via (at 106.4 134.9) (size 0.889) (layers F.Cu B.Cu) (net 20))
-  (segment (start 128 138) (end 128 136.4) (width 0.254) (layer B.Cu) (net 20))
-  (segment (start 128 136.4) (end 127.2 135.6) (width 0.254) (layer B.Cu) (net 20))
-  (segment (start 127.2 135.6) (end 124.9 135.6) (width 0.254) (layer B.Cu) (net 20))
-  (via (at 124.9 135.6) (size 0.889) (layers F.Cu B.Cu) (net 20))
-  (segment (start 124.9 135.6) (end 124.85 135.55) (width 0.254) (layer F.Cu) (net 20))
-  (segment (start 124.85 135.55) (end 118.5 135.55) (width 0.254) (layer F.Cu) (net 20))
+  (segment (start 106.4 134.9) (end 116.7 134.9) (width 0.254) (layer B.Cu) (net 20))
+  (via (at 116.7 134.9) (size 0.889) (layers F.Cu B.Cu) (net 20))
+  (segment (start 116.7 134.9) (end 117.35 135.55) (width 0.254) (layer F.Cu) (net 20))
+  (segment (start 117.35 135.55) (end 118.5 135.55) (width 0.254) (layer F.Cu) (net 20))
+  (segment (start 104.5 132) (end 104.5 129) (width 0.254) (layer F.Cu) (net 20))
+  (segment (start 104.5 129) (end 103.55 128.05) (width 0.254) (layer F.Cu) (net 20))
+  (segment (start 103 128.05) (end 103.55 128.05) (width 0.254) (layer F.Cu) (net 20))
+  (segment (start 104.5 133) (end 104.5 132) (width 0.254) (layer F.Cu) (net 20))
+  (segment (start 105.5 134) (end 104.5 133) (width 0.254) (layer F.Cu) (net 20))
   (segment (start 100.55 126.135) (end 102.815 126.135) (width 0.254) (layer F.Cu) (net 20))
   (segment (start 102.815 126.135) (end 103 125.95) (width 0.254) (layer F.Cu) (net 20))
@@
   (segment (start 125.95 126.8) (end 126.3 126.45) (width 0.254) (layer F.Cu) (net 20))
   (segment (start 118.5 135.55) (end 118.5 135.5) (width 0.254) (layer F.Cu) (net 20))
-  (segment (start 128 138) (end 128 136.5) (width 0.254) (layer F.Cu) (net 20))
-  (segment (start 129.5 131) (end 132 128.5) (width 0.254) (layer F.Cu) (net 20))
-  (segment (start 129.5 135) (end 129.5 131) (width 0.254) (layer F.Cu) (net 20))
-  (segment (start 128 136.5) (end 129.5 135) (width 0.254) (layer F.Cu) (net 20))
   (segment (start 106 132.45) (end 106.05 132.45) (width 0.254) (layer F.Cu) (net 21))
   (segment (start 118.35 131.5) (end 119.35 132.5) (width 0.254) (layer F.Cu) (net 21))
@@
   (segment (start 86.95 119.5) (end 86.95 117.5) (width 0.254) (layer F.Cu) (net 23))
   (segment (start 86.95 117.5) (end 87.85 116.6) (width 0.254) (layer F.Cu) (net 23))
+  (segment (start 118.5 137.45) (end 120.05 137.45) (width 0.254) (layer F.Cu) (net 24))
+  (via (at 120.5 137) (size 0.889) (layers F.Cu B.Cu) (net 24))
+  (segment (start 120.05 137.45) (end 120.5 137) (width 0.254) (layer F.Cu) (net 24))
   (segment (start 103.2 102.1) (end 103.9 101.4) (width 0.254) (layer F.Cu) (net 24))
   (segment (start 104.45 99.75) (end 103.9 100.3) (width 0.254) (layer F.Cu) (net 24))
@@
   (segment (start 134.6 130.3) (end 136.4 130.3) (width 0.254) (layer F.Cu) (net 46))
   (segment (start 132.4 132.5) (end 134.6 130.3) (width 0.254) (layer F.Cu) (net 46))
-  (segment (start 126 138) (end 126 133.85) (width 0.254) (layer F.Cu) (net 47))
-  (segment (start 126 133.85) (end 127.35 132.5) (width 0.254) (layer F.Cu) (net 47))
+  (segment (start 128 138) (end 128 133.15) (width 0.254) (layer F.Cu) (net 47))
+  (segment (start 128 133.15) (end 127.35 132.5) (width 0.254) (layer F.Cu) (net 47))
+  (segment (start 127.35 132.5) (end 127.5 132.5) (width 0.254) (layer F.Cu) (net 47))
+  (segment (start 127.5 132.5) (end 127.35 132.5) (width 0.254) (layer F.Cu) (net 47))
   (segment (start 123.65 132.5) (end 127.35 132.5) (width 0.254) (layer F.Cu) (net 47))
   (segment (start 114.5 120.55) (end 112.95 120.55) (width 0.254) (layer F.Cu) (net 48))
@@
     (polygon
       (pts
-        (xy 142.24 139.7) (xy 81.28 139.7) (xy 81.28 78.74) (xy 142.24 78.74)
+        (xy 140.97 138.43) (xy 82.55 138.43) (xy 82.55 80.01) (xy 140.97 80.01)
       )
     )
@@
     (polygon
       (pts
-        (xy 142.24 139.7) (xy 81.28 139.7) (xy 81.28 78.74) (xy 142.24 78.74)
+        (xy 140.97 138.43) (xy 82.55 138.43) (xy 82.55 80.01) (xy 140.97 80.01)
       )
     )
